Commit message: update mass and imu

File: rotors_description/urdf/component_snippets.xacro (robot description, xacro)
@@ -830,4 +830,24 @@
     </xacro:imu_plugin_macro>
   </xacro:macro>
+  <xacro:macro name="mpu6000_imu" params="namespace parent_link">
+    <!-- MPU6000 IMU -->
+    <xacro:imu_plugin_macro
+      namespace="${namespace}"
+      imu_suffix=""
+      parent_link="${parent_link}"
+      imu_topic="imu"
+      mass_imu_sensor="0.003"
+      gyroscope_noise_density="0.00008727"
+      gyroscope_random_walk="0.00000381"
+      gyroscope_bias_correlation_time="100.0"
+      gyroscope_turn_on_bias_sigma="0.00174"
+      accelerometer_noise_density="0.004"
+      accelerometer_random_walk="0.002"
+      accelerometer_bias_correlation_time="150.0"
+      accelerometer_turn_on_bias_sigma="0.0196">
+      <inertia ixx="0.000002" ixy="0.0" ixz="0.0" iyy="0.000002" iyz="0.0" izz="0.000002" />
+      <origin xyz="0 0 0" rpy="0 0 0" />
+    </xacro:imu_plugin_macro>
+</xacro:macro>
   <xacro:macro name="default_gps" params="namespace parent_link">
     <!-- Default GPS. -->
@@ -846,4 +866,21 @@
       <origin xyz="0 0 0" rpy="0 0 0" />
     </xacro:gps_plugin_macro>
+  </xacro:macro>
+  <xacro:macro name="fpv_gps" params="namespace parent_link">
+      <!-- Average GPS with 1m horizontal and 1m vertical position noise. -->
+      <xacro:gps_plugin_macro
+        namespace="${namespace}"
+        gps_suffix=""
+        parent_link="${parent_link}"
+        gps_topic="gps"
+        ground_speed_topic="ground_speed"
+        mass_gps_sensor="0.015"
+        horizontal_pos_std_dev="1.0"
+        vertical_pos_std_dev="1.0"
+        horizontal_vel_std_dev="0.1"
+        vertical_vel_std_dev="0.1">
+        <inertia ixx="0.00001" ixy="0.0" ixz="0.0" iyy="0.00001" iyz="0.0" izz="0.00001" />
+        <origin xyz="0 0 0" rpy="0 0 0" />
+      </xacro:gps_plugin_macro>
   </xacro:macro>
   <xacro:macro name="default_magnetometer" params="namespace parent_link">
